File: KiCAD/PCB Space.kicad_sch (KiCad schematic)
At the start: 10 parts, among them J1 Conn_01x03_Pin, U1 AP63300WU-7

Commit message: Poprawki + opis
Other:
- company: (none) -> Trytka Sp. z o.o.
Changed lines of the file:
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@@
 		(date "2026-10-26")
 		(rev "v2137")
+		(company "Trytka Sp. z o.o.")
 	)
 	(junction
